Commit message: fixed xacro tag

File: robosense_description/urdf/example.urdf.xacro (robot description, xacro)
@@ -2,22 +2,22 @@
 <robot xmlns:xacro="http://www.ros.org/wiki/xacro" name="example">
   <xacro:arg name="gpu" default="false"/>
-  <xacro:property name="gpu" value="$(arg gpu)" />
+  <xacro:property name="gpu" value="$(arg gpu)"/>
   <!-- Base Footprint -->
-  <link name="base_footprint" />
+  <link name="base_footprint"/>
   <!-- Base Link -->
-  <joint name="footprint" type="fixed" >
-   <parent link="base_footprint" />
-    <child link="base_link" />
-    <origin xyz="0 0 0.05" rpy="0 0 0" />
+  <joint name="footprint" type="fixed">
+    <parent link="base_footprint"/>
+    <child link="base_link"/>
+    <origin xyz="0 0 0.05" rpy="0 0 0"/>
   </joint>
-  <link name="base_link" >
+  <link name="base_link">
     <visual>
       <geometry>
-        <box size="0.5 0.5 0.1" />
+        <box size="0.5 0.5 0.1"/>
       </geometry>
     </visual>
     <collision>
       <geometry>
-        <box size="0.5 0.5 0.1" />
+        <box size="0.5 0.5 0.1"/>
       </geometry>
     </collision>
@@ -25,12 +25,10 @@
       <origin xyz="0 0 0"/>
       <mass value="10"/>
-      <inertia ixx="3.0" ixy="0.0" ixz="0.0"
-               iyy="3.0" iyz="0.0"
-               izz="3.0" />
+      <inertia ixx="3.0" ixy="0.0" ixz="0.0" iyy="3.0" iyz="0.0" izz="3.0"/>
     </inertial>
   </link>
   <xacro:include filename="$(find robosense_description)/urdf/RS-16.urdf.xacro"/>
-  <RS-16 parent="base_link" name="robosense" topic="/rs_points" hz="20" samples="900" gpu="${gpu}">
-    <origin xyz="0 0 0.4" rpy="0 0 0" />
-  </RS-16>
+  <xacro:RS-16 parent="base_link" name="robosense" topic="/rs_points" hz="20" samples="900" gpu="${gpu}">
+    <origin xyz="0 0 0.4" rpy="0 0 0"/>
+  </xacro:RS-16>
 </robot>
