Commit message: Added in channel 17 to 32 sensor.

File: robosense_description/urdf/RS-16.urdf.xacro (robot description, xacro)
@@ -1,8 +1,8 @@
 <?xml version="1.0"?>
 <robot xmlns:xacro="http://www.ros.org/wiki/xacro" name="RS-16">
-  <xacro:property name="M_PI" value="3.1415926535897931" />
+  <xacro:property name="M_PI" value="3.1415926535897931"/>
   <xacro:macro name="RS-16" params="*origin parent:=base_link name:=robosense topic:=/robosense_points hz:=20 lasers:=16 samples:=900 collision_range:=0.4 min_range:=0.4 max_range:=150.0 noise:=0.008 min_angle:=-${M_PI} max_angle:=${M_PI} gpu:=false">
     <joint name="${name}_base_mount_joint" type="fixed">
-      <xacro:insert_block name="origin" />
+      <xacro:insert_block name="origin"/>
       <parent link="${parent}"/>
       <child link="${name}_base_link"/>
@@ -12,12 +12,10 @@
         <mass value="0.87"/>
         <origin xyz="0 0 0"/>
-        <inertia ixx="0.001094695" ixy="0" ixz="0"
-          iyy="0.001094695" iyz="0"
-          izz="0.001245079"/>
+        <inertia ixx="0.001094695" ixy="0" ixz="0" iyy="0.001094695" iyz="0" izz="0.001245079"/>
       </inertial>
       <visual>
         <origin rpy="-1.5707 0 0" xyz="0 0 0"/>
         <geometry>
-          <mesh filename="package://robosense_description/meshes/robosense_16.dae" />
+          <mesh filename="package://robosense_description/meshes/robosense_16.dae"/>
         </geometry>
       </visual>
@@ -29,7 +27,7 @@
       </collision>
     </link>
-    <joint name="${name}_base_scan_joint" type="fixed" >
-      <origin xyz="0 0 0.039" rpy="0 0 0" />
-      <parent link="${name}_base_link" />
+    <joint name="${name}_base_scan_joint" type="fixed">
+      <origin xyz="0 0 0.039" rpy="0 0 0"/>
+      <parent link="${name}_base_link"/>
       <child link="${name}"/>
     </joint>
@@ -44,4 +42,5 @@
     <gazebo reference="${name}">
       <xacro:if value="${gpu}">
+        <!-- channnel 17 to 32. 3 deg increment. -->
         <sensor type="gpu_ray" name="${name}-RS16">
           <pose>0 0 0 0 0 0</pose>
@@ -57,8 +56,8 @@
               </horizontal>
               <vertical>
-                <samples>${lasers}</samples>
+                <samples>16</samples>
                 <resolution>1</resolution>
-                <min_angle>-${15.0*M_PI/180.0}</min_angle>
-                <max_angle> ${15.0*M_PI/180.0}</max_angle>
+                <min_angle>-${55*M_PI/180.0}</min_angle>
+                <max_angle>-${10*M_PI/180.0}</max_angle>
               </vertical>
             </scan>
@@ -100,5 +99,6 @@
                 <resolution>1</resolution>
                 <min_angle>-${15.0*M_PI/180.0}</min_angle>
-                <max_angle> ${15.0*M_PI/180.0}</max_angle>
+                <max_angle>
+                  ${15.0*M_PI/180.0}</max_angle>
               </vertical>
             </scan>

File: robosense_description/urdf/example.urdf.xacro (robot description, xacro)
@@ -29,6 +29,6 @@
   </link>
   <xacro:include filename="$(find robosense_description)/urdf/RS-16.urdf.xacro"/>
-  <xacro:RS-16 parent="base_link" name="robosense" topic="/rs_points" hz="20" samples="900" gpu="${gpu}">
-    <origin xyz="0 0 0.4" rpy="0 0 0"/>
+  <xacro:RS-16 parent="base_link" name="robosense" topic="/rs_points" hz="20" samples="900" gpu="true">
+    <origin xyz="0 0 1.4" rpy="0 0 0"/>
   </xacro:RS-16>
 </robot>

Commit message: first working macro for laserscan

File: robosense_description/urdf/RS-16.urdf.xacro (robot description, xacro)
@@ -8,5 +8,6 @@
       <child link="${name}_base_link"/>
     </joint>
-    <link name="${name}_base_link">
+    <!-- link for bottom of lidar -->
+    <link name="robosense_base_link">
       <inertial>
         <mass value="0.87"/>
@@ -27,101 +28,112 @@
       </collision>
     </link>
-    <joint name="${name}_base_scan_joint" type="fixed">
-      <origin xyz="0 0 0.039" rpy="0 0 0"/>
-      <parent link="${name}_base_link"/>
-      <child link="${name}"/>
-    </joint>
-    <link name="${name}">
-      <inertial>
-        <mass value="0.01"/>
-        <origin xyz="0 0 0"/>
-        <inertia ixx="1e-7" ixy="0" ixz="0" iyy="1e-7" iyz="0" izz="1e-7"/>
-      </inertial>
-    </link>
-    <!-- Gazebo requires the robosense_gazebo_plugins package -->
-    <gazebo reference="${name}">
-      <xacro:if value="${gpu}">
-        <!-- channnel 17 to 32. 3 deg increment. -->
-        <sensor type="gpu_ray" name="${name}-RS16">
-          <pose>0 0 0 0 0 0</pose>
-          <visualize>false</visualize>
-          <update_rate>${hz}</update_rate>
-          <ray>
-            <scan>
-              <horizontal>
-                <samples>${samples}</samples>
-                <resolution>1</resolution>
-                <min_angle>${min_angle}</min_angle>
-                <max_angle>${max_angle}</max_angle>
-              </horizontal>
-              <vertical>
-                <samples>16</samples>
-                <resolution>1</resolution>
-                <min_angle>-${55*M_PI/180.0}</min_angle>
-                <max_angle>-${10*M_PI/180.0}</max_angle>
-              </vertical>
-            </scan>
-            <range>
-              <min>${collision_range}</min>
-              <max>${max_range}</max>
-              <resolution>0.001</resolution>
-            </range>
-            <noise>
-              <type>gaussian</type>
-              <mean>0.0</mean>
-              <stddev>0.0</stddev>
-            </noise>
-          </ray>
-          <plugin name="gazebo_ros_laser_controller" filename="libgazebo_ros_robosense_gpu_laser.so">
-            <topicName>${topic}</topicName>
-            <frameName>${name}</frameName>
-            <min_range>${min_range}</min_range>
-            <max_range>${max_range}</max_range>
-            <gaussianNoise>${noise}</gaussianNoise>
-          </plugin>
-        </sensor>
-      </xacro:if>
-      <xacro:unless value="${gpu}">
-        <sensor type="ray" name="${name}-RS16">
-          <pose>0 0 0 0 0 0</pose>
-          <visualize>false</visualize>
-          <update_rate>${hz}</update_rate>
-          <ray>
-            <scan>
-              <horizontal>
-                <samples>${samples}</samples>
-                <resolution>1</resolution>
-                <min_angle>${min_angle}</min_angle>
-                <max_angle>${max_angle}</max_angle>
-              </horizontal>
-              <vertical>
-                <samples>${lasers}</samples>
-                <resolution>1</resolution>
-                <min_angle>-${15.0*M_PI/180.0}</min_angle>
-                <max_angle>
-                  ${15.0*M_PI/180.0}</max_angle>
-              </vertical>
-            </scan>
-            <range>
-              <min>${collision_range}</min>
-              <max>${max_range+1}</max>
-              <resolution>0.001</resolution>
-            </range>
-            <noise>
-              <type>gaussian</type>
-              <mean>0.0</mean>
-              <stddev>0.0</stddev>
-            </noise>
-          </ray>
-          <plugin name="gazebo_ros_laser_controller" filename="libgazebo_ros_robosense_laser.so">
-            <topicName>${topic}</topicName>
-            <frameName>${name}</frameName>
-            <min_range>${min_range}</min_range>
-            <max_range>${max_range}</max_range>
-            <gaussianNoise>${noise}</gaussianNoise>
-          </plugin>
-        </sensor>
-      </xacro:unless>
-    </gazebo>
+    <xacro:macro name="laserscan" params="name gpu hz min_angle max_angle vertmin vertmax samples layers topic collision_range max_range noise">
+      <joint name="${name}_base_scan_joint" type="fixed">
+        <origin xyz="0 0 0.039" rpy="0 0 0"/>
+        <parent link="robosense_base_link"/>
+        <child link="${name}"/>
+      </joint>
+      <!-- link for laserscan frame -->
+      <link name="${name}"/>
+      <!-- Gazebo requires the robosense_gazebo_plugins package -->
+      <gazebo reference="${name}">
+        <xacro:if value="${gpu}">
+          <!-- channnel 17 to 32. 3 deg increment. -->
+          <sensor type="gpu_ray" name="${name}-RS16">
+            <pose>0 0 0 0 0 0</pose>
+            <visualize>false</visualize>
+            <update_rate>${hz}</update_rate>
+            <ray>
+              <scan>
+                <horizontal>
+                  <samples>${samples}</samples>
+                  <resolution>1</resolution>
+                  <min_angle>${min_angle}</min_angle>
+                  <max_angle>${max_angle}</max_angle>
+                </horizontal>
+                <vertical>
+                  <samples>${layers}</samples>
+                  <resolution>1</resolution>
+                  <min_angle>${vertmin*M_PI/180.0}</min_angle>
+                  <max_angle>${vertmax*M_PI/180.0}</max_angle>
+                </vertical>
+              </scan>
+              <range>
+                <min>${collision_range}</min>
+                <max>${max_range}</max>
+                <resolution>0.001</resolution>
+              </range>
+              <noise>
+                <type>gaussian</type>
+                <mean>0.0</mean>
+                <stddev>0.0</stddev>
+              </noise>
+            </ray>
+            <plugin name="gazebo_ros_laser_controller" filename="libgazebo_ros_robosense_gpu_laser.so">
+              <topicName>${topic}</topicName>
+              <frameName>${name}</frameName>
+              <min_range>${min_range}</min_range>
+              <max_range>${max_range}</max_range>
+              <gaussianNoise>${noise}</gaussianNoise>
+            </plugin>
+          </sensor>
+        </xacro:if>
+        <xacro:unless value="${gpu}">
+          <sensor type="ray" name="${name}-RS16">
+            <pose>0 0 0 0 0 0</pose>
+            <visualize>false</visualize>
+            <update_rate>${hz}</update_rate>
+            <ray>
+              <scan>
+                <horizontal>
+                  <samples>${samples}</samples>
+                  <resolution>1</resolution>
+                  <min_angle>${min_angle}</min_angle>
+                  <max_angle>${max_angle}</max_angle>
+                </horizontal>
+                <vertical>
+                  <samples>${layers}</samples>
+                  <resolution>1</resolution>
+                  <min_angle>-${15.0*M_PI/180.0}</min_angle>
+                  <max_angle>
+                    ${15.0*M_PI/180.0}</max_angle>
+                </vertical>
+              </scan>
+              <range>
+                <min>${collision_range}</min>
+                <max>${max_range+1}</max>
+                <resolution>0.001</resolution>
+              </range>
+              <noise>
+                <type>gaussian</type>
+                <mean>0.0</mean>
+                <stddev>0.0</stddev>
+              </noise>
+            </ray>
+            <plugin name="gazebo_ros_laser_controller" filename="libgazebo_ros_robosense_laser.so">
+              <topicName>${topic}</topicName>
+              <frameName>${name}</frameName>
+              <min_range>${min_range}</min_range>
+              <max_range>${max_range}</max_range>
+              <gaussianNoise>${noise}</gaussianNoise>
+            </plugin>
+          </sensor>
+        </xacro:unless>
+      </gazebo>
+    </xacro:macro>
+    <xacro:laserscan
+      name="high"
+      gpu="${gpu}"
+      hz="${hz}"
+      min_angle="${min_angle}"
+      max_angle="${max_angle}"
+      vertmin="-55"
+      vertmax="-10"
+      samples="${samples}"
+      layers="16"
+      topic="yes"
+      collision_range="${collision_range}"
+      max_range="${max_range}"
+      noise="${noise}"/>
   </xacro:macro>
 </robot>

Commit message: removed unneccessary parameters.

File: robosense_description/urdf/RS-16.urdf.xacro (robot description, xacro)
@@ -28,5 +28,5 @@
       </collision>
     </link>
-    <xacro:macro name="laserscan" params="name gpu hz min_angle max_angle vertmin vertmax samples layers topic collision_range max_range noise">
+    <xacro:macro name="laserscan" params="name vertmin vertmax layers topic">
       <joint name="${name}_base_scan_joint" type="fixed">
         <origin xyz="0 0 0.039" rpy="0 0 0"/>
@@ -122,18 +122,5 @@
       </gazebo>
     </xacro:macro>
-    <xacro:laserscan
-      name="high"
-      gpu="${gpu}"
-      hz="${hz}"
-      min_angle="${min_angle}"
-      max_angle="${max_angle}"
-      vertmin="-55"
-      vertmax="-10"
-      samples="${samples}"
-      layers="16"
-      topic="yes"
-      collision_range="${collision_range}"
-      max_range="${max_range}"
-      noise="${noise}"/>
+    <xacro:laserscan name="high" vertmin="-55" vertmax="-10" layers="16" topic="yes"/>
   </xacro:macro>
 </robot>

Commit message: referenced all laserscans to one frame

File: robosense_description/urdf/RS-16.urdf.xacro (robot description, xacro)
@@ -28,17 +28,17 @@
       </collision>
     </link>
+    <!-- translation from base of lidar to the mid point of lidar -->
+    <joint name="${name}_base_scan_joint" type="fixed">
+      <origin xyz="0 0 0.039" rpy="0 0 0"/>
+      <parent link="robosense_base_link"/>
+      <child link="rslidar"/>
+    </joint>
+    <!-- main reference frame of all scans -->
+    <link name="rslidar"/>
     <xacro:macro name="laserscan" params="name vertmin vertmax layers topic">
-      <joint name="${name}_base_scan_joint" type="fixed">
-        <origin xyz="0 0 0.039" rpy="0 0 0"/>
-        <parent link="robosense_base_link"/>
-        <child link="${name}"/>
-      </joint>
-      <!-- link for laserscan frame -->
-      <link name="${name}"/>
       <!-- Gazebo requires the robosense_gazebo_plugins package -->
-      <gazebo reference="${name}">
+      <gazebo reference="rslidar">
         <xacro:if value="${gpu}">
-          <!-- channnel 17 to 32. 3 deg increment. -->
-          <sensor type="gpu_ray" name="${name}-RS16">
+          <sensor type="gpu_ray" name="${name}-5515">
             <pose>0 0 0 0 0 0</pose>
             <visualize>false</visualize>
@@ -72,5 +72,5 @@
             <plugin name="gazebo_ros_laser_controller" filename="libgazebo_ros_robosense_gpu_laser.so">
               <topicName>${topic}</topicName>
-              <frameName>${name}</frameName>
+              <frameName>rslidar</frameName>
               <min_range>${min_range}</min_range>
               <max_range>${max_range}</max_range>
@@ -112,5 +112,5 @@
             <plugin name="gazebo_ros_laser_controller" filename="libgazebo_ros_robosense_laser.so">
               <topicName>${topic}</topicName>
-              <frameName>${name}</frameName>
+              <frameName>rslidar</frameName>
               <min_range>${min_range}</min_range>
               <max_range>${max_range}</max_range>

Commit message: Removed unused parameters and tuned values.

File: robosense_description/urdf/RS-16.urdf.xacro (robot description, xacro)
@@ -2,5 +2,5 @@
 <robot xmlns:xacro="http://www.ros.org/wiki/xacro" name="RS-16">
   <xacro:property name="M_PI" value="3.1415926535897931"/>
-  <xacro:macro name="RS-16" params="*origin parent:=base_link name:=robosense topic:=/robosense_points hz:=20 lasers:=16 samples:=900 collision_range:=0.4 min_range:=0.4 max_range:=150.0 noise:=0.008 min_angle:=-${M_PI} max_angle:=${M_PI} gpu:=false">
+  <xacro:macro name="RS-16" params="*origin parent:=base_link name:=robosense hz:=10 samples:=1800 collision_range:=0.4 min_range:=0.1 max_range:=150.0 noise:=0.008 min_angle:=-${M_PI} max_angle:=${M_PI} gpu:=false">
     <joint name="${name}_base_mount_joint" type="fixed">
       <xacro:insert_block name="origin"/>

File: robosense_description/urdf/example.urdf.xacro (robot description, xacro)
@@ -29,5 +29,5 @@
   </link>
   <xacro:include filename="$(find robosense_description)/urdf/RS-16.urdf.xacro"/>
-  <xacro:RS-16 parent="base_link" name="robosense" topic="/rs_points" hz="20" samples="900" gpu="true">
+  <xacro:RS-16 parent="base_link" name="robosense" hz="10" samples="1800" gpu="true">
     <origin xyz="0 0 1.4" rpy="0 0 0"/>
   </xacro:RS-16>

Commit message: fixed lidar base naming issue

File: robosense_description/urdf/RS-16.urdf.xacro (robot description, xacro)
@@ -9,5 +9,5 @@
     </joint>
     <!-- link for bottom of lidar -->
-    <link name="robosense_base_link">
+    <link name="${name}_base_link">
       <inertial>
         <mass value="0.87"/>
@@ -31,5 +31,5 @@
     <joint name="${name}_base_scan_joint" type="fixed">
       <origin xyz="0 0 0.039" rpy="0 0 0"/>
-      <parent link="robosense_base_link"/>
+      <parent link="${name}_base_link"/>
       <child link="rslidar"/>
     </joint>

File: robosense_description/urdf/example.urdf.xacro (robot description, xacro)
@@ -29,5 +29,5 @@
   </link>
   <xacro:include filename="$(find robosense_description)/urdf/RS-16.urdf.xacro"/>
-  <xacro:RS-16 parent="base_link" name="robosense" hz="10" samples="1800" gpu="true">
+  <xacro:RS-16 parent="base_link" name="helios" hz="10" samples="1800" gpu="true">
     <origin xyz="0 0 1.4" rpy="0 0 0"/>
   </xacro:RS-16>

Commit message: updated translation

File: robosense_description/urdf/RS-16.urdf.xacro (robot description, xacro)
@@ -30,5 +30,5 @@
     <!-- translation from base of lidar to the mid point of lidar -->
     <joint name="${name}_base_scan_joint" type="fixed">
-      <origin xyz="0 0 0.039" rpy="0 0 0"/>
+      <origin xyz="0 0 0.050" rpy="0 0 0"/>
       <parent link="${name}_base_link"/>
       <child link="rslidar"/>
