Commit message: renamed files + scaled height

File: robosense_description/urdf/RS-5515.urdf.xacro (robot description, xacro)
@@ -1,6 +1,6 @@
 <?xml version="1.0"?>
-<robot xmlns:xacro="http://www.ros.org/wiki/xacro" name="RS-16">
+<robot xmlns:xacro="http://www.ros.org/wiki/xacro" name="RS-5515">
   <xacro:property name="M_PI" value="3.1415926535897931"/>
-  <xacro:macro name="RS-16" params="*origin parent:=base_link name:=robosense hz:=10 samples:=1800 collision_range:=0.4 min_range:=0.1 max_range:=150.0 noise:=0.008 min_angle:=-${M_PI} max_angle:=${M_PI} gpu:=false">
+  <xacro:macro name="RS-5515" params="*origin parent:=base_link name:=robosense hz:=10 samples:=1800 collision_range:=0.4 min_range:=0.1 max_range:=150.0 noise:=0.008 min_angle:=-${M_PI} max_angle:=${M_PI} gpu:=false">
     <joint name="${name}_base_mount_joint" type="fixed">
       <xacro:insert_block name="origin"/>

File: robosense_description/urdf/example.urdf.xacro (robot description, xacro)
@@ -28,7 +28,7 @@
     </inertial>
   </link>
-  <xacro:include filename="$(find robosense_description)/urdf/RS-16.urdf.xacro"/>
-  <xacro:RS-16 parent="base_link" name="helios" hz="10" samples="1800" gpu="true">
-    <origin xyz="0 0 1.4" rpy="0 0 0"/>
-  </xacro:RS-16>
+  <xacro:include filename="$(find robosense_description)/urdf/RS-5515.urdf.xacro"/>
+  <xacro:RS-5515 parent="base_link" name="helios" hz="10" samples="1800" gpu="true">
+    <origin xyz="0 0 1.35" rpy="0 0 0"/>
+  </xacro:RS-5515>
 </robot>

Commit message: Added in a cylinder to represent the lidar

File: robosense_description/urdf/RS-5515.urdf.xacro (robot description, xacro)
@@ -16,13 +16,13 @@
       </inertial>
       <visual>
-        <origin rpy="-1.5707 0 0" xyz="0 0 0"/>
+        <origin rpy="0 0 0" xyz="0 0 0.05"/>
         <geometry>
-          <mesh filename="package://robosense_description/meshes/robosense_16.dae"/>
+          <cylinder radius="0.05" length="0.1"/>
         </geometry>
       </visual>
       <collision>
-        <origin rpy="0 0 0" xyz="0 0 0"/>
+        <origin rpy="0 0 0" xyz="0 0 0.05"/>
         <geometry>
-          <cylinder radius="0.0535" length="0.0817"/>
+          <cylinder radius="0.05" length="0.1"/>
         </geometry>
       </collision>

Commit message: reduced default noise level and added pclmerger into example launch file

File: robosense_description/urdf/RS-5515.urdf.xacro (robot description, xacro)
@@ -2,5 +2,5 @@
 <robot xmlns:xacro="http://www.ros.org/wiki/xacro" name="RS-5515">
   <xacro:property name="M_PI" value="3.1415926535897931"/>
-  <xacro:macro name="RS-5515" params="*origin parent:=base_link name:=robosense hz:=10 samples:=1800 collision_range:=0.4 min_range:=0.1 max_range:=150.0 noise:=0.008 min_angle:=-${M_PI} max_angle:=${M_PI} gpu:=false">
+  <xacro:macro name="RS-5515" params="*origin parent:=base_link name:=robosense hz:=10 samples:=1800 collision_range:=0.4 min_range:=0.1 max_range:=150.0 noise:=0.002 min_angle:=-${M_PI} max_angle:=${M_PI} gpu:=false">
     <joint name="${name}_base_mount_joint" type="fixed">
       <xacro:insert_block name="origin"/>

File: robosense_description/urdf/example.urdf.xacro (robot description, xacro)
@@ -29,5 +29,9 @@
   </link>
   <xacro:include filename="$(find robosense_description)/urdf/RS-5515.urdf.xacro"/>
-  <xacro:RS-5515 parent="base_link" name="helios" hz="10" samples="1800" gpu="true">
+  <!-- hz: scan rate of lidar. -->
+  <!-- samples: no. of points in a horizontal plane. -->
+  <!-- gpu: true to use gpu to compute pointcloud-->
+  <!-- noise: a greater value would result in more sensor noise -->
+  <xacro:RS-5515 parent="base_link" name="helios" hz="10" samples="1800" gpu="true" noise="0.002">
     <origin xyz="0 0 1.35" rpy="0 0 0"/>
   </xacro:RS-5515>

Commit message: removed intertia tag

File: robosense_description/urdf/RS-5515.urdf.xacro (robot description, xacro)
@@ -10,9 +10,4 @@
     <!-- link for bottom of lidar -->
     <link name="${name}_base_link">
-      <inertial>
-        <mass value="0.87"/>
-        <origin xyz="0 0 0"/>
-        <inertia ixx="0.001094695" ixy="0" ixz="0" iyy="0.001094695" iyz="0" izz="0.001245079"/>
-      </inertial>
       <visual>
         <origin rpy="0 0 0" xyz="0 0 0.05"/>
